File: ALIMENTACIONKICAD/alimentacion.kicad_sch (KiCad schematic)
At the start: 20 parts, among them J1 Conn_01x02_Male, J2 Conn_01x02_Male, J4 Conn_01x02_Male, U1 MIC29302WT, U2 SPX3819M5-L-3-3, U4 MIC5219-3.3YM5

Commit message: hola
Parts:
- removed C1: 100u, symbol Device:C_Polarized_Small_US
- removed C10, C5, C7: 10u, symbol Device:C
- removed C11: 0.1u, symbol Device:C
- removed C2: 1u, Capacitor_SMD:C_0603_1608Metric_Pad1.08x0.95mm_HandSolder, symbol Device:C
- removed C3: 330u, symbol Device:C_Polarized_Small_US
- removed C4: 100n, symbol Device:C
- removed C6: 1u, symbol Device:C_Polarized
- removed J1, J2, J4: Conn_01x02_Male, symbol Connector:Conn_01x02_Male
- removed R1: 100k, symbol Device:R
- removed R2: 43k, symbol Device:R
- removed R3: 470, symbol Device:R
- removed R4, R5: R, symbol Device:R
- removed U1: MIC29302WT, Package_TO_SOT_THT:TO-220-5_P3.4x3.7mm_StaggerEven_Lead3.8mm_Vertical, symbol Regulator_Linear:MIC29302WT
- removed U2: SPX3819M5-L-3-3, Package_TO_SOT_SMD:SOT-23-5, symbol Regulator_Linear:SPX3819M5-L-3-3
- removed U4: MIC5219-3.3YM5, Package_TO_SOT_SMD:SOT-23-5, symbol Regulator_Linear:MIC5219-3.3YM5
- added C?: 330u, symbol Device:C_Polarized_Small_US
- added C?: 100n, symbol Device:C
- added C?: 1u, symbol Device:C_Polarized
- added C? (x3): 10u, symbol Device:C
- added C?: 1u, Capacitor_SMD:C_0603_1608Metric_Pad1.08x0.95mm_HandSolder, symbol Device:C
- added C?: 0.1u, symbol Device:C
- added C?: 100u, symbol Device:C_Polarized_Small_US
- added J? (x3): Conn_01x02_Male, symbol Connector:Conn_01x02_Male
- added R? (x2): R, symbol Device:R
- added R?: 470, symbol Device:R
- added R?: 100k, symbol Device:R
- added R?: 43k, symbol Device:R
- added U?: SPX3819M5-L-3-3, Package_TO_SOT_SMD:SOT-23-5, symbol Regulator_Linear:SPX3819M5-L-3-3
- added U?: MIC29302WT, Package_TO_SOT_THT:TO-220-5_P3.4x3.7mm_StaggerEven_Lead3.8mm_Vertical, symbol Regulator_Linear:MIC29302WT
- added U?: MIC5219-3.3YM5, Package_TO_SOT_SMD:SOT-23-5, symbol Regulator_Linear:MIC5219-3.3YM5
Connections:
- net +3.3V: now also C?.1, C?.1, C?.1, R?.1, U?.5 (OUT), U?.5 (OUT)
- net +5V: now also C?.1, C?.1, J?.1 (Pin_1), U?.2 (VIN)
- net 4.1V: now also C?.1, C?.1, R?.1, R?.1, U?.4 (VOUT)
- net Esp32: now also U?.1 (EN), U?.3 (EN), U?.3 (EN)
- net GND: now also C?.2, C?.2, C?.2, C?.2, C?.2, C?.2, C?.2, C?.2, C?.2, J?.2 (Pin_2), J?.2 (Pin_2), J?.2 (Pin_2), R?.2, R?.2, R?.2, U?.2 (GND), U?.2 (GND), U?.3 (GND)
- new net: R?.1, R?.2
- new net: C?.1, J?.1 (Pin_1), U?.1 (IN)
- new net: J?.1 (Pin_1), U?.1 (IN)
- new net: C?.1, U?.4 (BP)
- new net: R?.1, R?.2, U?.5 (ADJ)
