File: Embebidos/alimentacion/alimentacion.kicad_sch (KiCad schematic)
At the start: 24 parts, among them J1 Conn_01x02_Male, J2 Conn_01x02_Male, J3 Conn_01x02_Male, J4 Conn_01x02_Male, U1 MIC29302WT, U2 SPX3819M5-L-3-3, U3 AMS1117-3.3, U4 MIC5219-3.3YM5

Commit message: modificado
Parts:
- removed C8, C9: 10u, symbol Device:C
- removed J3: Conn_01x02_Male, symbol Connector:Conn_01x02_Male
- removed U3: AMS1117-3.3, Package_TO_SOT_SMD:SOT-223-3_TabPin2, symbol Regulator_Linear:AMS1117-3.3
