File: Embebidos/LDR-module.kicad_sch (KiCad schematic)
At the start: 12 parts

Commit message: Corrección de anotaciones
Parts:
- gave numbers to parts that had none: 10
Changed lines of the file:
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@@
   (symbol (lib_id "Device:R") (at 144.78 43.18 0) (unit 1)
     (in_bom yes) (on_board yes) (fields_autoplaced)
-    (property "Reference" "R?" (id 0) (at 147.32 41.9099 0)
+    (property "Reference" "R17" (id 0) (at 147.32 41.9099 0)
       (effects (font (size 1.27 1.27)) (justify left))
     )
@@
   (symbol (lib_id "power:GND") (at 55.88 67.31 0) (unit 1)
     (in_bom yes) (on_board yes) (fields_autoplaced)
-    (property "Reference" "#PWR?" (id 0) (at 55.88 73.66 0)
+    (property "Reference" "#PWR018" (id 0) (at 55.88 73.66 0)
       (effects (font (size 1.27 1.27)) hide)
     )
@@
   (symbol (lib_id "Amplifier_Operational:LM358") (at 134.62 59.69 0) (mirror x) (unit 1)
     (in_bom yes) (on_board yes) (fields_autoplaced)
-    (property "Reference" "U?" (id 0) (at 134.62 49.53 0))
+    (property "Reference" "U2" (id 0) (at 134.62 49.53 0))
     (property "Value" "LM358" (id 1) (at 134.62 52.07 0))
     (property "Footprint" "" (id 2) (at 134.62 59.69 0)
@@
   (symbol (lib_id "power:GND") (at 116.84 54.61 0) (unit 1)
     (in_bom yes) (on_board yes) (fields_autoplaced)
-    (property "Reference" "#PWR?" (id 0) (at 116.84 60.96 0)
+    (property "Reference" "#PWR021" (id 0) (at 116.84 60.96 0)
       (effects (font (size 1.27 1.27)) hide)
     )
@@
   (symbol (lib_id "Amplifier_Operational:LM358") (at 134.62 78.74 0) (unit 2)
     (in_bom yes) (on_board yes) (fields_autoplaced)
-    (property "Reference" "U?" (id 0) (at 134.62 68.58 0))
+    (property "Reference" "U2" (id 0) (at 134.62 68.58 0))
     (property "Value" "LM358" (id 1) (at 134.62 71.12 0))
     (property "Footprint" "" (id 2) (at 134.62 78.74 0)
@@
   (symbol (lib_id "Device:R") (at 68.58 54.61 0) (unit 1)
     (in_bom yes) (on_board yes) (fields_autoplaced)
-    (property "Reference" "R?" (id 0) (at 71.12 53.3399 0)
+    (property "Reference" "R14" (id 0) (at 71.12 53.3399 0)
       (effects (font (size 1.27 1.27)) (justify left))
     )
@@
   (symbol (lib_id "Amplifier_Operational:LM358") (at 58.42 57.15 0) (unit 3)
     (in_bom yes) (on_board yes) (fields_autoplaced)
-    (property "Reference" "U?" (id 0) (at 57.15 55.8799 0)
+    (property "Reference" "U2" (id 0) (at 57.15 55.8799 0)
       (effects (font (size 1.27 1.27)) (justify left))
     )
@@
   (symbol (lib_id "Device:R_Potentiometer") (at 116.84 48.26 0) (unit 1)
     (in_bom yes) (on_board yes) (fields_autoplaced)
-    (property "Reference" "RV?" (id 0) (at 114.3 46.9899 0)
+    (property "Reference" "RV1" (id 0) (at 114.3 46.9899 0)
       (effects (font (size 1.27 1.27)) (justify right))
     )
@@
   (symbol (lib_id "Sensor_Optical:LDR07") (at 96.52 67.31 0) (unit 1)
     (in_bom yes) (on_board yes) (fields_autoplaced)
-    (property "Reference" "R?" (id 0) (at 99.06 66.0399 0)
+    (property "Reference" "R16" (id 0) (at 99.06 66.0399 0)
       (effects (font (size 1.27 1.27)) (justify left))
     )
@@
   (symbol (lib_id "Device:LED") (at 144.78 53.34 90) (unit 1)
     (in_bom yes) (on_board yes) (fields_autoplaced)
-    (property "Reference" "D?" (id 0) (at 148.59 53.6574 90)
+    (property "Reference" "D4" (id 0) (at 148.59 53.6574 90)
       (effects (font (size 1.27 1.27)) (justify right))
     )
@@
   (symbol (lib_id "Device:R") (at 96.52 54.61 0) (unit 1)
     (in_bom yes) (on_board yes) (fields_autoplaced)
-    (property "Reference" "R?" (id 0) (at 99.06 53.3399 0)
+    (property "Reference" "R15" (id 0) (at 99.06 53.3399 0)
       (effects (font (size 1.27 1.27)) (justify left))
     )
@@
   (symbol (lib_id "power:+5V") (at 55.88 46.99 0) (unit 1)
     (in_bom yes) (on_board yes) (fields_autoplaced)
-    (property "Reference" "#PWR?" (id 0) (at 55.88 50.8 0)
+    (property "Reference" "#PWR017" (id 0) (at 55.88 50.8 0)
       (effects (font (size 1.27 1.27)) hide)
     )
@@
   (symbol (lib_id "power:GND") (at 90.17 77.47 0) (unit 1)
     (in_bom yes) (on_board yes) (fields_autoplaced)
-    (property "Reference" "#PWR?" (id 0) (at 90.17 83.82 0)
+    (property "Reference" "#PWR020" (id 0) (at 90.17 83.82 0)
       (effects (font (size 1.27 1.27)) hide)
     )
@@
   (symbol (lib_id "power:+5V") (at 90.17 35.56 0) (unit 1)
     (in_bom yes) (on_board yes) (fields_autoplaced)
-    (property "Reference" "#PWR?" (id 0) (at 90.17 39.37 0)
+    (property "Reference" "#PWR019" (id 0) (at 90.17 39.37 0)
       (effects (font (size 1.27 1.27)) hide)
     )
@@
   (symbol (lib_id "Device:C_Small") (at 82.55 60.96 0) (unit 1)
     (in_bom yes) (on_board yes) (fields_autoplaced)
-    (property "Reference" "C?" (id 0) (at 85.09 59.6962 0)
+    (property "Reference" "C8" (id 0) (at 85.09 59.6962 0)
       (effects (font (size 1.27 1.27)) (justify left))
     )
@@
   (symbol (lib_id "Device:C_Small") (at 107.95 67.31 0) (unit 1)
     (in_bom yes) (on_board yes) (fields_autoplaced)
-    (property "Reference" "C?" (id 0) (at 110.49 66.0462 0)
+    (property "Reference" "C9" (id 0) (at 110.49 66.0462 0)
       (effects (font (size 1.27 1.27)) (justify left))
     )
@@
   (symbol (lib_id "Device:LED") (at 68.58 67.31 90) (unit 1)
     (in_bom yes) (on_board yes)
-    (property "Reference" "D?" (id 0) (at 71.12 67.31 90)
-      (effects (font (size 1.27 1.27)) (justify right))
-    )
+    (property "Reference" "D3" (id 0) (at 71.12 67.31 90)
+      (effects (font (size 1.27 1.27)) (justify right))
+    )
