File: Embebidos/LDR-module.kicad_sch (KiCad schematic)
At the start: 10 parts, among them U2 LM358

Commit message: Huellas
Parts:
- C8, C9: value 104 -> 0.1u
- RV1: footprint (none) -> Potentiometer_THT:Potentiometer_Bourns_3386P_Vertical
Changed lines of the file:
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@@
       (effects (font (size 1.27 1.27)) (justify right))
     )
-    (property "Footprint" "" (id 2) (at 116.84 48.26 0)
+    (property "Footprint" "Potentiometer_THT:Potentiometer_Bourns_3386P_Vertical" (id 2) (at 116.84 48.26 0)
       (effects (font (size 1.27 1.27)) hide)
     )
@@
       (effects (font (size 1.27 1.27)) (justify left))
     )
-    (property "Value" "104" (id 1) (at 85.09 62.2362 0)
+    (property "Value" "0.1u" (id 1) (at 85.09 62.2362 0)
       (effects (font (size 1.27 1.27)) (justify left))
     )
@@
       (effects (font (size 1.27 1.27)) (justify left))
     )
-    (property "Value" "104" (id 1) (at 110.49 68.5862 0)
+    (property "Value" "0.1u" (id 1) (at 110.49 68.5862 0)
       (effects (font (size 1.27 1.27)) (justify left))
     )
