File: Embebidos/EsquemaGeneral.kicad_sch (KiCad schematic)
At the start: 0 parts

Commit message: LDR_69Errores
Other:
- sheet Acondicionamiento ports: added LDR_IN; removed none
Changed lines of the file:
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@@
+    (stroke (width 0) (type default) (color 0 0 0 0))
+  )
+  (wire (pts (xy 31.75 22.86) (xy 24.13 22.86))
     (stroke (width 0) (type default) (color 0 0 0 0))
   )
@@
     (stroke (width 0) (type default) (color 0 0 0 0))
   )
+  (wire (pts (xy 24.13 44.45) (xy 31.75 44.45))
+    (stroke (width 0) (type default) (color 0 0 0 0))
+  )
   (wire (pts (xy 76.2 59.69) (xy 88.9 59.69))
     (stroke (width 0) (type default) (color 0 0 0 0))
@@
     (stroke (width 0) (type default) (color 0 0 0 0))
   )
+  (wire (pts (xy 24.13 22.86) (xy 24.13 44.45))
+    (stroke (width 0) (type default) (color 0 0 0 0))
+  )
   (wire (pts (xy 76.2 82.55) (xy 139.7 82.55))
     (stroke (width 0) (type default) (color 0 0 0 0))
@@
     )
   )
-  (sheet (at 154.94 38.1) (size 13.97 11.43) (fields_autoplaced)
-    (stroke (width 0.1524) (type solid) (color 0 0 0 0))
-    (fill (color 0 0 0 0.0000))
-    (property "Sheet name" "LDR-module" (id 0) (at 154.94 37.3884 0)
-      (effects (font (size 1.27 1.27)) (justify left bottom))
-    )
-    (property "Sheet file" "LDR-module.kicad_sch" (id 1) (at 154.94 50.1146 0)
-      (effects (font (size 1.27 1.27)) (justify left top))
-    )
-    (pin "DOUT" output (at 154.94 40.64 180)
+  (sheet (at 31.75 20.32) (size 13.97 11.43) (fields_autoplaced)
+    (stroke (width 0.1524) (type solid) (color 0 0 0 0))
+    (fill (color 0 0 0 0.0000))
+    (property "Sheet name" "LDR-module" (id 0) (at 31.75 19.6084 0)
+      (effects (font (size 1.27 1.27)) (justify left bottom))
+    )
+    (property "Sheet file" "LDR-module.kicad_sch" (id 1) (at 31.75 32.3346 0)
+      (effects (font (size 1.27 1.27)) (justify left top))
+    )
+    (pin "DOUT" output (at 31.75 22.86 180)
       (effects (font (size 1.27 1.27)) (justify left))
     )
@@
       (effects (font (size 1.27 1.27)) (justify left))
     )
+    (pin "LDR_IN" input (at 31.75 44.45 180)
+      (effects (font (size 1.27 1.27)) (justify left))
+    )
