File: Embebidos/Luces_traseras2.kicad_sch (KiCad schematic)
At the start: 8 parts, among them J8 RJ45, Q5 BSS138, Q6 DMP3056LSDQ-13

Commit message: Huellas
Parts:
- J8: footprint (none) -> Connector_RJ:RJ45_Amphenol_54602-x08_Horizontal
- R25, R26, R27, R28, R29: footprint (none) -> Resistor_SMD:R_0805_2012Metric_Pad1.20x1.40mm_HandSolder
Changed lines of the file:
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@@
     (property "Reference" "R28" (id 0) (at 55.88 78.5622 90))
     (property "Value" "470" (id 1) (at 55.88 80.8736 90))
-    (property "Footprint" "" (id 2) (at 55.88 82.042 90)
+    (property "Footprint" "Resistor_SMD:R_0805_2012Metric_Pad1.20x1.40mm_HandSolder" (id 2) (at 55.88 82.042 90)
       (effects (font (size 1.27 1.27)) hide)
     )
@@
     (property "Reference" "R29" (id 0) (at 63.5 99.06 90))
     (property "Value" "470" (id 1) (at 63.5 101.3714 90))
-    (property "Footprint" "" (id 2) (at 63.5 94.742 90)
+    (property "Footprint" "Resistor_SMD:R_0805_2012Metric_Pad1.20x1.40mm_HandSolder" (id 2) (at 63.5 94.742 90)
       (effects (font (size 1.27 1.27)) hide)
     )
@@
       (effects (font (size 1.27 1.27)) (justify right))
     )
-    (property "Footprint" "" (id 2) (at 111.76 92.075 90)
+    (property "Footprint" "Connector_RJ:RJ45_Amphenol_54602-x08_Horizontal" (id 2) (at 111.76 92.075 90)
       (effects (font (size 1.27 1.27)) hide)
     )
@@
     (property "Reference" "R25" (id 0) (at 31.75 147.32 90))
     (property "Value" "1k" (id 1) (at 31.75 149.86 90))
-    (property "Footprint" "" (id 2) (at 31.75 151.638 90)
+    (property "Footprint" "Resistor_SMD:R_0805_2012Metric_Pad1.20x1.40mm_HandSolder" (id 2) (at 31.75 151.638 90)
       (effects (font (size 1.27 1.27)) hide)
     )
@@
     (property "Reference" "R27" (id 0) (at 45.72 137.16 90))
     (property "Value" "100k" (id 1) (at 48.26 137.16 90))
-    (property "Footprint" "" (id 2) (at 50.038 137.16 90)
+    (property "Footprint" "Resistor_SMD:R_0805_2012Metric_Pad1.20x1.40mm_HandSolder" (id 2) (at 50.038 137.16 90)
       (effects (font (size 1.27 1.27)) hide)
     )
@@
     (property "Reference" "R26" (id 0) (at 35.56 156.21 90))
     (property "Value" "100k" (id 1) (at 38.1 156.21 90))
-    (property "Footprint" "" (id 2) (at 39.878 156.21 90)
+    (property "Footprint" "Resistor_SMD:R_0805_2012Metric_Pad1.20x1.40mm_HandSolder" (id 2) (at 39.878 156.21 90)
       (effects (font (size 1.27 1.27)) hide)
     )

Commit message: Anotaciones
Parts:
- renumbered J8 to J4
Changed lines of the file:
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@@
   (symbol (lib_id "Connector:RJ45") (at 111.76 91.44 180) (unit 1)
     (in_bom yes) (on_board yes)
-    (property "Reference" "J8" (id 0) (at 120.142 91.5416 0)
+    (property "Reference" "J4" (id 0) (at 120.142 91.5416 0)
       (effects (font (size 1.27 1.27)) (justify right))
     )
