File: Embebidos/alimentacion.kicad_sch (KiCad schematic)
At the start: 18 parts, among them J2 Conn_01x02_Male, U3 SPX3819M5-L-3-3, U4 MIC29302WT, U5 MIC5219-3.3YM5

Commit message: ajustes
Parts:
- added C111: 1u, symbol Device:C
- C10: value 10u -> 10n
- C13: value 1u -> 4.7u
- C15: value 10u -> 1u
- C17: value 10u -> 470p
- C18: value 0.1u -> 2.2u
Connections:
- net +5V: now also C111.1
- net 3.3Vop2: no longer C17.1
- net GND: now also C111.2
- net at U5.4 (BP): now also C17.1
- no-connect marks 1 -> 0
Other:
- note added: "Alimentacion con regulador de 3.3V para la ESP32. GPS las R sobran se pueden usar para regular Estados del EN (ON>2V) (OFF<0.4V)"
- note added: "Alimentacion de 3.3V LDR RFID se deja un regulador separado para poder controlar el funcionamiento de algunos modulos sin desactivar la alimentacion de la ESP32 C18 Tantalum"
- note removed: "Alimentacion con regulador de 3.3V para la ESP32. las R sobran se pueden usar para regular"
- note removed: "Alimentacion de 3.3V GPS LDR RFID se deja un regulador separado para poder controlar el funcionamiento de algunos modulos sin desactivar la alimentacion de la ESP32"
Changed lines of the file:
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@@
   (junction (at 99.695 160.02) (diameter 0) (color 0 0 0 0)
   )
+  (junction (at 33.02 68.58) (diameter 0) (color 0 0 0 0)
+  )
   (junction (at 52.705 139.065) (diameter 0) (color 0 0 0 0)
   )
@@
   (junction (at 132.715 139.065) (diameter 0) (color 0 0 0 0)
   )
+  (junction (at 45.72 81.28) (diameter 0) (color 0 0 0 0)
+  )
   (junction (at 162.56 97.79) (diameter 0) (color 0 0 0 0)
   )
@@
   (junction (at 77.47 66.04) (diameter 0) (color 0 0 0 0)
   )
-  (junction (at 182.88 81.28) (diameter 0) (color 0 0 0 0)
-  )
   (junction (at 132.715 160.02) (diameter 0) (color 0 0 0 0)
   )
@@
   (junction (at 61.595 139.065) (diameter 0) (color 0 0 0 0)
   )
-  (no_connect (at 170.18 83.82))
   (wire (pts (xy 195.58 90.17) (xy 195.58 81.28))
     (stroke (width 0) (type default) (color 0 0 0 0))
@@
     (stroke (width 0) (type default) (color 0 0 0 0))
   )
+  (wire (pts (xy 33.02 81.28) (xy 45.72 81.28))
+    (stroke (width 0) (type default) (color 0 0 0 0))
+  )
+  (wire (pts (xy 33.02 78.74) (xy 33.02 81.28))
+    (stroke (width 0) (type default) (color 0 0 0 0))
+  )
   (wire (pts (xy 33.02 63.5) (xy 33.02 66.04))
     (stroke (width 0) (type default) (color 0 0 0 0))
@@
     (stroke (width 0) (type default) (color 0 0 0 0))
   )
-  (wire (pts (xy 182.88 90.17) (xy 182.88 81.28))
-    (stroke (width 0) (type default) (color 0 0 0 0))
-  )
   (wire (pts (xy 99.695 160.02) (xy 114.3 160.02))
     (stroke (width 0) (type default) (color 0 0 0 0))
@@
     (stroke (width 0) (type default) (color 0 0 0 0))
   )
-  (wire (pts (xy 195.58 81.28) (xy 182.88 81.28))
+  (wire (pts (xy 170.18 81.28) (xy 195.58 81.28))
+    (stroke (width 0) (type default) (color 0 0 0 0))
+  )
+  (wire (pts (xy 170.18 83.82) (xy 182.88 83.82))
     (stroke (width 0) (type default) (color 0 0 0 0))
   )
@@
     (stroke (width 0) (type default) (color 0 0 0 0))
   )
-  (wire (pts (xy 182.88 81.28) (xy 170.18 81.28))
-    (stroke (width 0) (type default) (color 0 0 0 0))
-  )
-  (wire (pts (xy 45.72 76.2) (xy 45.72 85.09))
+  (wire (pts (xy 45.72 76.2) (xy 45.72 81.28))
     (stroke (width 0) (type default) (color 0 0 0 0))
   )
@@
     (stroke (width 0) (type default) (color 0 0 0 0))
   )
+  (wire (pts (xy 33.02 68.58) (xy 33.02 71.12))
+    (stroke (width 0) (type default) (color 0 0 0 0))
+  )
   (wire (pts (xy 67.31 74.93) (xy 67.31 78.74))
     (stroke (width 0) (type default) (color 0 0 0 0))
@@
     (stroke (width 0) (type default) (color 0 0 0 0))
   )
+  (wire (pts (xy 45.72 81.28) (xy 45.72 85.09))
+    (stroke (width 0) (type default) (color 0 0 0 0))
+  )
+  (wire (pts (xy 182.88 83.82) (xy 182.88 90.17))
+    (stroke (width 0) (type default) (color 0 0 0 0))
+  )
   (wire (pts (xy 132.715 139.065) (xy 132.715 144.145))
     (stroke (width 0) (type default) (color 0 0 0 0))
@@
     (stroke (width 0) (type default) (color 0 0 0 0))
   )
-  (text "Alimentacion de 3.3V\nGPS\nLDR\nRFID\nse deja un regulador\nseparado para poder controlar\nel funcionamiento de algunos modulos\nsin desactivar la alimentacion de la ESP32\n"
+  (text "Alimentacion de 3.3V\nLDR\nRFID\nse deja un regulador\nseparado para poder controlar\nel funcionamiento de algunos modulos\nsin desactivar la alimentacion de la ESP32\nC18 Tantalum\n"
     (at 212.09 105.41 0)
     (effects (font (size 1.27 1.27)) (justify left bottom))
@@
     (effects (font (size 1.27 1.27)) (justify left bottom))
   )
-  (text "Alimentacion con regulador de 3.3V \npara la ESP32.\nlas R sobran se pueden usar para regular\n"
-    (at 27.94 105.41 0)
+  (text "Alimentacion con regulador de 3.3V \npara la ESP32. GPS\nlas R sobran se pueden usar para regular\nEstados del EN (ON>2V) (OFF<0.4V)\n"
+    (at 26.67 106.68 0)
     (effects (font (size 1.27 1.27)) (justify left bottom))
   )
@@
       (effects (font (size 1.27 1.27)) (justify left))
     )
-    (property "Value" "10u" (id 1) (at 143.51 88.8999 0)
+    (property "Value" "1u" (id 1) (at 143.51 88.8999 0)
       (effects (font (size 1.27 1.27)) (justify left))
     )
@@
     (pin "1")
   )
+  (symbol (lib_id "Device:C") (at 33.02 74.93 0) (unit 1)
+    (in_bom yes) (on_board yes) (fields_autoplaced)
+    (property "Reference" "C111" (id 0) (at 36.83 73.6599 0)
+      (effects (font (size 1.27 1.27)) (justify left))
+    )
+    (property "Value" "1u" (id 1) (at 36.83 76.1999 0)
+      (effects (font (size 1.27 1.27)) (justify left))
+    )
+    (property "Footprint" "" (id 2) (at 33.9852 78.74 0)
+      (effects (font (size 1.27 1.27)) hide)
+    )
+    (property "Datasheet" "~" (id 3) (at 33.02 74.93 0)
+      (effects (font (size 1.27 1.27)) hide)
+    )
+    (pin "1")
+    (pin "2")
+  )
   (symbol (lib_id "Device:C") (at 143.51 146.685 0) (unit 1)
     (in_bom yes) (on_board yes)
@@
       (effects (font (size 1.27 1.27)) (justify left))
     )
-    (property "Value" "0.1u" (id 1) (at 199.39 95.2499 0)
+    (property "Value" "2.2u" (id 1) (at 199.39 95.2499 0)
       (effects (font (size 1.27 1.27)) (justify left))
     )
@@
       (effects (font (size 1.27 1.27)) (justify left))
     )
-    (property "Value" "10u" (id 1) (at 60.96 74.9299 0)
+    (property "Value" "10n" (id 1) (at 60.96 74.9299 0)
       (effects (font (size 1.27 1.27)) (justify left))
     )
@@
       (effects (font (size 1.27 1.27)) (justify left))
     )
-    (property "Value" "10u" (id 1) (at 186.69 95.2499 0)
+    (property "Value" "470p" (id 1) (at 186.69 95.2499 0)
       (effects (font (size 1.27 1.27)) (justify left))
     )
@@
       (effects (font (size 1.27 1.27)) (justify left))
     )
-    (property "Value" "1u" (id 1) (at 81.28 72.7709 0)
-      (effects (font (size 1.27 1.27)) (justify left))
-    )
+    (property "Value" "4.7u" (id 1) (at 81.28 72.7709 0)
+      (effects (font (size 1.27 1.27)) (justify left))
+    )

Commit message: noseuwu
Parts:
- removed R19, R20: R, symbol Device:R
- C111: footprint (none) -> Capacitor_SMD:C_0805_2012Metric_Pad1.18x1.45mm_HandSolder
Other:
- moved on the sheet: C13
Changed lines of the file:
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@@
   (junction (at 61.595 160.02) (diameter 0) (color 0 0 0 0)
   )
-  (junction (at 77.47 66.04) (diameter 0) (color 0 0 0 0)
+  (junction (at 67.31 66.04) (diameter 0) (color 0 0 0 0)
   )
   (junction (at 132.715 160.02) (diameter 0) (color 0 0 0 0)
   )
-  (junction (at 67.31 66.04) (diameter 0) (color 0 0 0 0)
-  )
   (junction (at 95.885 160.02) (diameter 0) (color 0 0 0 0)
   )
@@
     (stroke (width 0) (type default) (color 0 0 0 0))
   )
-  (wire (pts (xy 67.31 86.36) (xy 67.31 90.17))
-    (stroke (width 0) (type default) (color 0 0 0 0))
-  )
   (wire (pts (xy 38.1 68.58) (xy 33.02 68.58))
     (stroke (width 0) (type default) (color 0 0 0 0))
@@
     (stroke (width 0) (type default) (color 0 0 0 0))
   )
-  (polyline (pts (xy 87.63 53.34) (xy 87.63 99.06))
+  (polyline (pts (xy 77.47 53.34) (xy 77.47 99.06))
     (stroke (width 0) (type default) (color 0 0 0 0))
   )
@@
     (stroke (width 0) (type default) (color 0 0 0 0))
   )
-  (wire (pts (xy 77.47 66.04) (xy 77.47 68.58))
+  (wire (pts (xy 67.31 66.04) (xy 67.31 68.58))
     (stroke (width 0) (type default) (color 0 0 0 0))
   )
@@
     (stroke (width 0) (type default) (color 0 0 0 0))
   )
-  (polyline (pts (xy 87.63 99.06) (xy 27.94 99.06))
+  (polyline (pts (xy 77.47 99.06) (xy 27.94 99.06))
     (stroke (width 0) (type default) (color 0 0 0 0))
   )
@@
     (stroke (width 0) (type default) (color 0 0 0 0))
   )
-  (wire (pts (xy 77.47 76.2) (xy 77.47 78.74))
+  (wire (pts (xy 67.31 76.2) (xy 67.31 78.74))
     (stroke (width 0) (type default) (color 0 0 0 0))
   )
@@
     (stroke (width 0) (type default) (color 0 0 0 0))
   )
-  (wire (pts (xy 77.47 64.77) (xy 77.47 66.04))
+  (wire (pts (xy 67.31 64.77) (xy 67.31 66.04))
     (stroke (width 0) (type default) (color 0 0 0 0))
   )
@@
     (stroke (width 0) (type default) (color 0 0 0 0))
   )
-  (wire (pts (xy 67.31 66.04) (xy 67.31 67.31))
-    (stroke (width 0) (type default) (color 0 0 0 0))
-  )
   (wire (pts (xy 61.595 139.065) (xy 52.705 139.065))
     (stroke (width 0) (type default) (color 0 0 0 0))
   )
-  (wire (pts (xy 77.47 66.04) (xy 67.31 66.04))
-    (stroke (width 0) (type default) (color 0 0 0 0))
-  )
   (wire (pts (xy 139.7 81.28) (xy 154.94 81.28))
     (stroke (width 0) (type default) (color 0 0 0 0))
@@
     (stroke (width 0) (type default) (color 0 0 0 0))
   )
-  (wire (pts (xy 67.31 74.93) (xy 67.31 78.74))
-    (stroke (width 0) (type default) (color 0 0 0 0))
-  )
   (wire (pts (xy 42.545 160.02) (xy 61.595 160.02))
     (stroke (width 0) (type default) (color 0 0 0 0))
@@
     (stroke (width 0) (type default) (color 0 0 0 0))
   )
-  (polyline (pts (xy 27.94 53.34) (xy 87.63 53.34))
+  (polyline (pts (xy 27.94 53.34) (xy 77.47 53.34))
     (stroke (width 0) (type default) (color 0 0 0 0))
   )
@@
   )
   (text "Alimentacion de 3.3V\nLDR\nRFID\nse deja un regulador\nseparado para poder controlar\nel funcionamiento de algunos modulos\nsin desactivar la alimentacion de la ESP32\nC18 Tantalum\n"
-    (at 212.09 105.41 0)
+    (at 209.55 107.95 0)
     (effects (font (size 1.27 1.27)) (justify left bottom))
   )
-  (text "Alimentacion con regulador a 4.1V \nusado para alimentar unicamente el\nmodulo SIM\n\n>Pin enable requiere aproximadamente 20uA"
+  (text "Alimentacion con regulador a 4.1V \nusado para alimentar unicamente el\nmodulo SIM\n>Pin enable requiere aproximadamente 20uA"
     (at 24.13 172.72 0)
     (effects (font (size 1.27 1.27)) (justify left bottom))
   )
   (text "Alimentacion con regulador de 3.3V \npara la ESP32. GPS\nlas R sobran se pueden usar para regular\nEstados del EN (ON>2V) (OFF<0.4V)\n"
-    (at 26.67 106.68 0)
+    (at 27.94 107.95 0)
     (effects (font (size 1.27 1.27)) (justify left bottom))
   )
@@
     (pin "1")
     (pin "2")
-  )
-  (symbol (lib_id "power:GND") (at 67.31 90.17 0) (unit 1)
-    (in_bom yes) (on_board yes) (fields_autoplaced)
-    (property "Reference" "#PWR025" (id 0) (at 67.31 96.52 0)
-      (effects (font (size 1.27 1.27)) hide)
-    )
-    (property "Value" "GND" (id 1) (at 67.31 95.25 0))
-    (property "Footprint" "" (id 2) (at 67.31 90.17 0)
-      (effects (font (size 1.27 1.27)) hide)
-    )
-    (property "Datasheet" "" (id 3) (at 67.31 90.17 0)
-      (effects (font (size 1.27 1.27)) hide)
-    )
-    (pin "1")
   )
   (symbol (lib_id "Regulator_Linear:MIC29302WT") (at 95.885 141.605 0) (unit 1)
@@
       (effects (font (size 1.27 1.27)) (justify left))
     )
-    (property "Footprint" "" (id 2) (at 33.9852 78.74 0)
+    (property "Footprint" "Capacitor_SMD:C_0805_2012Metric_Pad1.18x1.45mm_HandSolder" (id 2) (at 33.9852 78.74 0)
       (effects (font (size 1.27 1.27)) hide)
     )
@@
     (pin "5")
   )
-  (symbol (lib_id "Device:R") (at 67.31 71.12 0) (unit 1)
-    (in_bom yes) (on_board yes) (fields_autoplaced)
-    (property "Reference" "R19" (id 0) (at 69.85 69.8499 0)
-      (effects (font (size 1.27 1.27)) (justify left))
-    )
-    (property "Value" "R" (id 1) (at 69.85 72.3899 0)
-      (effects (font (size 1.27 1.27)) (justify left))
-    )
-    (property "Footprint" "" (id 2) (at 65.532 71.12 90)
-      (effects (font (size 1.27 1.27)) hide)
-    )
-    (property "Datasheet" "~" (id 3) (at 67.31 71.12 0)
-      (effects (font (size 1.27 1.27)) hide)
-    )
-    (pin "1")
-    (pin "2")
-  )
-  (symbol (lib_id "power:GND") (at 77.47 78.74 0) (unit 1)
-    (in_bom yes) (on_board yes) (fields_autoplaced)
-    (property "Reference" "#PWR027" (id 0) (at 77.47 85.09 0)
-      (effects (font (size 1.27 1.27)) hide)
-    )
-    (property "Value" "GND" (id 1) (at 77.47 83.82 0))
-    (property "Footprint" "" (id 2) (at 77.47 78.74 0)
-      (effects (font (size 1.27 1.27)) hide)
-    )
-    (property "Datasheet" "" (id 3) (at 77.47 78.74 0)
-      (effects (font (size 1.27 1.27)) hide)
-    )
-    (pin "1")
-  )
-  (symbol (lib_id "power:+3.3V") (at 77.47 64.77 0) (unit 1)
+  (symbol (lib_id "power:GND") (at 67.31 78.74 0) (unit 1)
+    (in_bom yes) (on_board yes) (fields_autoplaced)
+    (property "Reference" "#PWR027" (id 0) (at 67.31 85.09 0)
+      (effects (font (size 1.27 1.27)) hide)
+    )
+    (property "Value" "GND" (id 1) (at 67.31 83.82 0))
+    (property "Footprint" "" (id 2) (at 67.31 78.74 0)
+      (effects (font (size 1.27 1.27)) hide)
+    )
+    (property "Datasheet" "" (id 3) (at 67.31 78.74 0)
+      (effects (font (size 1.27 1.27)) hide)
+    )
+    (pin "1")
+  )
+  (symbol (lib_id "power:+3.3V") (at 67.31 64.77 0) (unit 1)
     (in_bom yes) (on_board yes)
-    (property "Reference" "#PWR026" (id 0) (at 77.47 68.58 0)
-      (effects (font (size 1.27 1.27)) hide)
-    )
-    (property "Value" "+3.3V" (id 1) (at 77.851 60.3758 0))
-    (property "Footprint" "" (id 2) (at 77.47 64.77 0)
-      (effects (font (size 1.27 1.27)) hide)
-    )
-    (property "Datasheet" "" (id 3) (at 77.47 64.77 0)
-      (effects (font (size 1.27 1.27)) hide)
-    )
-    (pin "1")
-  )
-  (symbol (lib_id "Device:R") (at 67.31 82.55 0) (unit 1)
-    (in_bom yes) (on_board yes) (fields_autoplaced)
-    (property "Reference" "R20" (id 0) (at 69.85 81.2799 0)
-      (effects (font (size 1.27 1.27)) (justify left))
-    )
-    (property "Value" "R" (id 1) (at 69.85 83.8199 0)
-      (effects (font (size 1.27 1.27)) (justify left))
-    )
-    (property "Footprint" "" (id 2) (at 65.532 82.55 90)
-      (effects (font (size 1.27 1.27)) hide)
-    )
-    (property "Datasheet" "~" (id 3) (at 67.31 82.55 0)
-      (effects (font (size 1.27 1.27)) hide)
-    )
-    (pin "1")
-    (pin "2")
+    (property "Reference" "#PWR026" (id 0) (at 67.31 68.58 0)
+      (effects (font (size 1.27 1.27)) hide)
+    )
+    (property "Value" "+3.3V" (id 1) (at 67.691 60.3758 0))
+    (property "Footprint" "" (id 2) (at 67.31 64.77 0)
+      (effects (font (size 1.27 1.27)) hide)
+    )
+    (property "Datasheet" "" (id 3) (at 67.31 64.77 0)
+      (effects (font (size 1.27 1.27)) hide)
+    )
+    (pin "1")
   )
   (symbol (lib_id "power:GND") (at 45.72 85.09 0) (unit 1)
@@
   )
   (symbol (lib_id "Device:C") (at 57.15 73.66 0) (unit 1)
-    (in_bom yes) (on_board yes) (fields_autoplaced)
-    (property "Reference" "C10" (id 0) (at 60.96 72.3899 0)
-      (effects (font (size 1.27 1.27)) (justify left))
-    )
-    (property "Value" "10n" (id 1) (at 60.96 74.9299 0)
+    (in_bom yes) (on_board yes)
+    (property "Reference" "C10" (id 0) (at 58.42 71.12 0)
+      (effects (font (size 1.27 1.27)) (justify left))
+    )
+    (property "Value" "10n" (id 1) (at 58.42 76.2 0)
       (effects (font (size 1.27 1.27)) (justify left))
     )
@@
     (pin "2")
   )
-  (symbol (lib_id "Device:C_Polarized") (at 77.47 72.39 0) (unit 1)
-    (in_bom yes) (on_board yes) (fields_autoplaced)
-    (property "Reference" "C13" (id 0) (at 81.28 70.2309 0)
-      (effects (font (size 1.27 1.27)) (justify left))
-    )
-    (property "Value" "4.7u" (id 1) (at 81.28 72.7709 0)
-      (effects (font (size 1.27 1.27)) (justify left))
-    )
-    (property "Footprint" "" (id 2) (at 78.4352 76.2 0)
-      (effects (font (size 1.27 1.27)) hide)
-    )
-    (property "Datasheet" "~" (id 3) (at 77.47 72.39 0)
-      (effects (font (size 1.27 1.27)) hide)
-    )
+  (symbol (lib_id "Device:C_Polarized") (at 67.31 72.39 0) (unit 1)
+    (in_bom yes) (on_board yes) (fields_autoplaced)
+    (property "Reference" "C13" (id 0) (at 71.12 70.2309 0)
+      (effects (font (size 1.27 1.27)) (justify left))
+    )
+    (property "Value" "4.7u" (id 1) (at 71.12 72.7709 0)
+      (effects (font (size 1.27 1.27)) (justify left))
+    )
+    (property "Footprint" "" (id 2) (at 68.2752 76.2 0)
+      (effects (font (size 1.27 1.27)) hide)
+    )
+    (property "Datasheet" "~" (id 3) (at 67.31 72.39 0)
+      (effects (font (size 1.27 1.27)) hide)
+    )

Commit message: r33
Parts:
- renumbered C111 to C10, C10 to C11, C11 to C12, C12 to C14, C14 to C15, C15 to C16, C16 to C17, C17 to C18, C18 to C19, R21 to R19, R22 to R20, R23 to R21
Changed lines of the file:
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@@
   (symbol (lib_id "Device:C") (at 139.7 87.63 0) (unit 1)
     (in_bom yes) (on_board yes) (fields_autoplaced)
-    (property "Reference" "C15" (id 0) (at 143.51 86.3599 0)
+    (property "Reference" "C16" (id 0) (at 143.51 86.3599 0)
       (effects (font (size 1.27 1.27)) (justify left))
     )
@@
   (symbol (lib_id "power:GND") (at 57.15 80.01 0) (unit 1)
     (in_bom yes) (on_board yes) (fields_autoplaced)
-    (property "Reference" "#PWR024" (id 0) (at 57.15 86.36 0)
+    (property "Reference" "#PWR025" (id 0) (at 57.15 86.36 0)
       (effects (font (size 1.27 1.27)) hide)
     )
@@
   (symbol (lib_id "Device:C") (at 33.02 74.93 0) (unit 1)
     (in_bom yes) (on_board yes) (fields_autoplaced)
-    (property "Reference" "C111" (id 0) (at 36.83 73.6599 0)
+    (property "Reference" "C10" (id 0) (at 36.83 73.6599 0)
       (effects (font (size 1.27 1.27)) (justify left))
     )
@@
   (symbol (lib_id "Device:C") (at 143.51 146.685 0) (unit 1)
     (in_bom yes) (on_board yes)
-    (property "Reference" "C16" (id 0) (at 147.32 145.4149 0)
+    (property "Reference" "C17" (id 0) (at 147.32 145.4149 0)
       (effects (font (size 1.27 1.27)) (justify left))
     )
@@
   (symbol (lib_id "Device:C") (at 195.58 93.98 0) (unit 1)
     (in_bom yes) (on_board yes) (fields_autoplaced)
-    (property "Reference" "C18" (id 0) (at 199.39 92.7099 0)
+    (property "Reference" "C19" (id 0) (at 199.39 92.7099 0)
       (effects (font (size 1.27 1.27)) (justify left))
     )
@@
   (symbol (lib_id "Device:C") (at 73.025 145.415 0) (unit 1)
     (in_bom yes) (on_board yes) (fields_autoplaced)
-    (property "Reference" "C12" (id 0) (at 76.835 144.1449 0)
+    (property "Reference" "C14" (id 0) (at 76.835 144.1449 0)
       (effects (font (size 1.27 1.27)) (justify left))
     )
@@
   (symbol (lib_id "Device:R") (at 114.3 145.415 0) (unit 1)
     (in_bom yes) (on_board yes) (fields_autoplaced)
-    (property "Reference" "R21" (id 0) (at 116.84 144.1449 0)
+    (property "Reference" "R19" (id 0) (at 116.84 144.1449 0)
       (effects (font (size 1.27 1.27)) (justify left))
     )
@@
   (symbol (lib_id "Device:R") (at 153.035 147.32 0) (unit 1)
     (in_bom yes) (on_board yes)
-    (property "Reference" "R23" (id 0) (at 155.575 146.0499 0)
+    (property "Reference" "R21" (id 0) (at 155.575 146.0499 0)
       (effects (font (size 1.27 1.27)) (justify left))
     )
@@
   (symbol (lib_id "power:GND") (at 45.72 85.09 0) (unit 1)
     (in_bom yes) (on_board yes) (fields_autoplaced)
-    (property "Reference" "#PWR022" (id 0) (at 45.72 91.44 0)
+    (property "Reference" "#PWR023" (id 0) (at 45.72 91.44 0)
       (effects (font (size 1.27 1.27)) hide)
     )
@@
   (symbol (lib_id "Device:R") (at 114.3 154.94 0) (unit 1)
     (in_bom yes) (on_board yes) (fields_autoplaced)
-    (property "Reference" "R22" (id 0) (at 116.84 153.6699 0)
+    (property "Reference" "R20" (id 0) (at 116.84 153.6699 0)
       (effects (font (size 1.27 1.27)) (justify left))
     )
@@
   (symbol (lib_id "Device:C_Polarized_Small_US") (at 132.715 146.685 0) (unit 1)
     (in_bom yes) (on_board yes)
-    (property "Reference" "C14" (id 0) (at 135.89 144.9831 0)
+    (property "Reference" "C15" (id 0) (at 135.89 144.9831 0)
       (effects (font (size 1.27 1.27)) (justify left))
     )
@@
   (symbol (lib_id "Device:C") (at 57.15 73.66 0) (unit 1)
     (in_bom yes) (on_board yes)
-    (property "Reference" "C10" (id 0) (at 58.42 71.12 0)
+    (property "Reference" "C11" (id 0) (at 58.42 71.12 0)
       (effects (font (size 1.27 1.27)) (justify left))
     )
@@
   (symbol (lib_id "Device:C_Polarized_Small_US") (at 61.595 145.415 0) (unit 1)
     (in_bom yes) (on_board yes)
-    (property "Reference" "C11" (id 0) (at 64.77 143.7131 0)
+    (property "Reference" "C12" (id 0) (at 64.77 143.7131 0)
       (effects (font (size 1.27 1.27)) (justify left))
     )
@@
   (symbol (lib_id "power:+5V") (at 33.02 63.5 0) (unit 1)
     (in_bom yes) (on_board yes) (fields_autoplaced)
-    (property "Reference" "#PWR021" (id 0) (at 33.02 67.31 0)
+    (property "Reference" "#PWR022" (id 0) (at 33.02 67.31 0)
       (effects (font (size 1.27 1.27)) hide)
     )
@@
   (symbol (lib_id "Device:C") (at 182.88 93.98 0) (unit 1)
     (in_bom yes) (on_board yes) (fields_autoplaced)
-    (property "Reference" "C17" (id 0) (at 186.69 92.7099 0)
+    (property "Reference" "C18" (id 0) (at 186.69 92.7099 0)
       (effects (font (size 1.27 1.27)) (justify left))
     )
@@
   (symbol (lib_id "power:+5V") (at 52.705 137.795 0) (unit 1)
     (in_bom yes) (on_board yes) (fields_autoplaced)
-    (property "Reference" "#PWR023" (id 0) (at 52.705 141.605 0)
-      (effects (font (size 1.27 1.27)) hide)
-    )
+    (property "Reference" "#PWR024" (id 0) (at 52.705 141.605 0)
+      (effects (font (size 1.27 1.27)) hide)
+    )
