File: Embebidos/alimentacion.kicad_sch (KiCad schematic)
At the start: 17 parts, among them J2 Conn_01x02_Male, U3 SPX3819M5-L-3-3, U4 MIC29302WT, U5 MIC5219-3.3YM5

Commit message: nosex2
Parts:
- C13: footprint (none) -> Capacitor_Tantalum_SMD:CP_EIA-6032-15_Kemet-U_Pad2.25x2.35mm_HandSolder
- renumbered C11 to C10, C12 to C11, C10 to C111, C14 to C12, C15 to C14, C16 to C15, C17 to C16, C18 to C17, C19 to C18, R19 to R21, R20 to R22, R21 to R23
Changed lines of the file:
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@@
   (symbol (lib_id "Device:C") (at 139.7 87.63 0) (unit 1)
     (in_bom yes) (on_board yes) (fields_autoplaced)
-    (property "Reference" "C16" (id 0) (at 143.51 86.3599 0)
+    (property "Reference" "C15" (id 0) (at 143.51 86.3599 0)
       (effects (font (size 1.27 1.27)) (justify left))
     )
@@
   (symbol (lib_id "power:GND") (at 57.15 80.01 0) (unit 1)
     (in_bom yes) (on_board yes) (fields_autoplaced)
-    (property "Reference" "#PWR025" (id 0) (at 57.15 86.36 0)
+    (property "Reference" "#PWR024" (id 0) (at 57.15 86.36 0)
       (effects (font (size 1.27 1.27)) hide)
     )
@@
   (symbol (lib_id "Device:C") (at 33.02 74.93 0) (unit 1)
     (in_bom yes) (on_board yes) (fields_autoplaced)
-    (property "Reference" "C10" (id 0) (at 36.83 73.6599 0)
+    (property "Reference" "C111" (id 0) (at 36.83 73.6599 0)
       (effects (font (size 1.27 1.27)) (justify left))
     )
@@
   (symbol (lib_id "Device:C") (at 143.51 146.685 0) (unit 1)
     (in_bom yes) (on_board yes)
-    (property "Reference" "C17" (id 0) (at 147.32 145.4149 0)
+    (property "Reference" "C16" (id 0) (at 147.32 145.4149 0)
       (effects (font (size 1.27 1.27)) (justify left))
     )
@@
   (symbol (lib_id "Device:C") (at 195.58 93.98 0) (unit 1)
     (in_bom yes) (on_board yes) (fields_autoplaced)
-    (property "Reference" "C19" (id 0) (at 199.39 92.7099 0)
+    (property "Reference" "C18" (id 0) (at 199.39 92.7099 0)
       (effects (font (size 1.27 1.27)) (justify left))
     )
@@
   (symbol (lib_id "Device:C") (at 73.025 145.415 0) (unit 1)
     (in_bom yes) (on_board yes) (fields_autoplaced)
-    (property "Reference" "C14" (id 0) (at 76.835 144.1449 0)
+    (property "Reference" "C12" (id 0) (at 76.835 144.1449 0)
       (effects (font (size 1.27 1.27)) (justify left))
     )
@@
   (symbol (lib_id "Device:R") (at 114.3 145.415 0) (unit 1)
     (in_bom yes) (on_board yes) (fields_autoplaced)
-    (property "Reference" "R19" (id 0) (at 116.84 144.1449 0)
+    (property "Reference" "R21" (id 0) (at 116.84 144.1449 0)
       (effects (font (size 1.27 1.27)) (justify left))
     )
@@
   (symbol (lib_id "Device:R") (at 153.035 147.32 0) (unit 1)
     (in_bom yes) (on_board yes)
-    (property "Reference" "R21" (id 0) (at 155.575 146.0499 0)
+    (property "Reference" "R23" (id 0) (at 155.575 146.0499 0)
       (effects (font (size 1.27 1.27)) (justify left))
     )
@@
   (symbol (lib_id "power:GND") (at 45.72 85.09 0) (unit 1)
     (in_bom yes) (on_board yes) (fields_autoplaced)
-    (property "Reference" "#PWR023" (id 0) (at 45.72 91.44 0)
+    (property "Reference" "#PWR022" (id 0) (at 45.72 91.44 0)
       (effects (font (size 1.27 1.27)) hide)
     )
@@
   (symbol (lib_id "Device:R") (at 114.3 154.94 0) (unit 1)
     (in_bom yes) (on_board yes) (fields_autoplaced)
-    (property "Reference" "R20" (id 0) (at 116.84 153.6699 0)
+    (property "Reference" "R22" (id 0) (at 116.84 153.6699 0)
       (effects (font (size 1.27 1.27)) (justify left))
     )
@@
   (symbol (lib_id "Device:C_Polarized_Small_US") (at 132.715 146.685 0) (unit 1)
     (in_bom yes) (on_board yes)
-    (property "Reference" "C15" (id 0) (at 135.89 144.9831 0)
+    (property "Reference" "C14" (id 0) (at 135.89 144.9831 0)
       (effects (font (size 1.27 1.27)) (justify left))
     )
@@
   (symbol (lib_id "Device:C") (at 57.15 73.66 0) (unit 1)
     (in_bom yes) (on_board yes)
-    (property "Reference" "C11" (id 0) (at 58.42 71.12 0)
+    (property "Reference" "C10" (id 0) (at 58.42 71.12 0)
       (effects (font (size 1.27 1.27)) (justify left))
     )
@@
   (symbol (lib_id "Device:C_Polarized_Small_US") (at 61.595 145.415 0) (unit 1)
     (in_bom yes) (on_board yes)
-    (property "Reference" "C12" (id 0) (at 64.77 143.7131 0)
+    (property "Reference" "C11" (id 0) (at 64.77 143.7131 0)
       (effects (font (size 1.27 1.27)) (justify left))
     )
@@
   (symbol (lib_id "power:+5V") (at 33.02 63.5 0) (unit 1)
     (in_bom yes) (on_board yes) (fields_autoplaced)
-    (property "Reference" "#PWR022" (id 0) (at 33.02 67.31 0)
+    (property "Reference" "#PWR021" (id 0) (at 33.02 67.31 0)
       (effects (font (size 1.27 1.27)) hide)
     )
@@
   (symbol (lib_id "Device:C") (at 182.88 93.98 0) (unit 1)
     (in_bom yes) (on_board yes) (fields_autoplaced)
-    (property "Reference" "C18" (id 0) (at 186.69 92.7099 0)
+    (property "Reference" "C17" (id 0) (at 186.69 92.7099 0)
       (effects (font (size 1.27 1.27)) (justify left))
     )
@@
       (effects (font (size 1.27 1.27)) (justify left))
     )
-    (property "Footprint" "" (id 2) (at 68.2752 76.2 0)
+    (property "Footprint" "Capacitor_Tantalum_SMD:CP_EIA-6032-15_Kemet-U_Pad2.25x2.35mm_HandSolder" (id 2) (at 68.2752 76.2 0)
       (effects (font (size 1.27 1.27)) hide)
     )
@@
   (symbol (lib_id "power:+5V") (at 52.705 137.795 0) (unit 1)
     (in_bom yes) (on_board yes) (fields_autoplaced)
-    (property "Reference" "#PWR024" (id 0) (at 52.705 141.605 0)
-      (effects (font (size 1.27 1.27)) hide)
-    )
+    (property "Reference" "#PWR023" (id 0) (at 52.705 141.605 0)
+      (effects (font (size 1.27 1.27)) hide)
+    )

Commit message: fpesp
Parts:
- renumbered C111 to C10, C10 to C11, C11 to C12, C12 to C14, C14 to C15, C15 to C16, C16 to C17, C17 to C18, C18 to C19, R21 to R19, R22 to R20, R23 to R21
Changed lines of the file:
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@@
   (symbol (lib_id "Device:C") (at 139.7 87.63 0) (unit 1)
     (in_bom yes) (on_board yes) (fields_autoplaced)
-    (property "Reference" "C15" (id 0) (at 143.51 86.3599 0)
+    (property "Reference" "C16" (id 0) (at 143.51 86.3599 0)
       (effects (font (size 1.27 1.27)) (justify left))
     )
@@
   (symbol (lib_id "power:GND") (at 57.15 80.01 0) (unit 1)
     (in_bom yes) (on_board yes) (fields_autoplaced)
-    (property "Reference" "#PWR024" (id 0) (at 57.15 86.36 0)
+    (property "Reference" "#PWR025" (id 0) (at 57.15 86.36 0)
       (effects (font (size 1.27 1.27)) hide)
     )
@@
   (symbol (lib_id "Device:C") (at 33.02 74.93 0) (unit 1)
     (in_bom yes) (on_board yes) (fields_autoplaced)
-    (property "Reference" "C111" (id 0) (at 36.83 73.6599 0)
+    (property "Reference" "C10" (id 0) (at 36.83 73.6599 0)
       (effects (font (size 1.27 1.27)) (justify left))
     )
@@
   (symbol (lib_id "Device:C") (at 143.51 146.685 0) (unit 1)
     (in_bom yes) (on_board yes)
-    (property "Reference" "C16" (id 0) (at 147.32 145.4149 0)
+    (property "Reference" "C17" (id 0) (at 147.32 145.4149 0)
       (effects (font (size 1.27 1.27)) (justify left))
     )
@@
   (symbol (lib_id "Device:C") (at 195.58 93.98 0) (unit 1)
     (in_bom yes) (on_board yes) (fields_autoplaced)
-    (property "Reference" "C18" (id 0) (at 199.39 92.7099 0)
+    (property "Reference" "C19" (id 0) (at 199.39 92.7099 0)
       (effects (font (size 1.27 1.27)) (justify left))
     )
@@
   (symbol (lib_id "Device:C") (at 73.025 145.415 0) (unit 1)
     (in_bom yes) (on_board yes) (fields_autoplaced)
-    (property "Reference" "C12" (id 0) (at 76.835 144.1449 0)
+    (property "Reference" "C14" (id 0) (at 76.835 144.1449 0)
       (effects (font (size 1.27 1.27)) (justify left))
     )
@@
   (symbol (lib_id "Device:R") (at 114.3 145.415 0) (unit 1)
     (in_bom yes) (on_board yes) (fields_autoplaced)
-    (property "Reference" "R21" (id 0) (at 116.84 144.1449 0)
+    (property "Reference" "R19" (id 0) (at 116.84 144.1449 0)
       (effects (font (size 1.27 1.27)) (justify left))
     )
@@
   (symbol (lib_id "Device:R") (at 153.035 147.32 0) (unit 1)
     (in_bom yes) (on_board yes)
-    (property "Reference" "R23" (id 0) (at 155.575 146.0499 0)
+    (property "Reference" "R21" (id 0) (at 155.575 146.0499 0)
       (effects (font (size 1.27 1.27)) (justify left))
     )
@@
   (symbol (lib_id "power:GND") (at 45.72 85.09 0) (unit 1)
     (in_bom yes) (on_board yes) (fields_autoplaced)
-    (property "Reference" "#PWR022" (id 0) (at 45.72 91.44 0)
+    (property "Reference" "#PWR023" (id 0) (at 45.72 91.44 0)
       (effects (font (size 1.27 1.27)) hide)
     )
@@
   (symbol (lib_id "Device:R") (at 114.3 154.94 0) (unit 1)
     (in_bom yes) (on_board yes) (fields_autoplaced)
-    (property "Reference" "R22" (id 0) (at 116.84 153.6699 0)
+    (property "Reference" "R20" (id 0) (at 116.84 153.6699 0)
       (effects (font (size 1.27 1.27)) (justify left))
     )
@@
   (symbol (lib_id "Device:C_Polarized_Small_US") (at 132.715 146.685 0) (unit 1)
     (in_bom yes) (on_board yes)
-    (property "Reference" "C14" (id 0) (at 135.89 144.9831 0)
+    (property "Reference" "C15" (id 0) (at 135.89 144.9831 0)
       (effects (font (size 1.27 1.27)) (justify left))
     )
@@
   (symbol (lib_id "Device:C") (at 57.15 73.66 0) (unit 1)
     (in_bom yes) (on_board yes)
-    (property "Reference" "C10" (id 0) (at 58.42 71.12 0)
+    (property "Reference" "C11" (id 0) (at 58.42 71.12 0)
       (effects (font (size 1.27 1.27)) (justify left))
     )
@@
   (symbol (lib_id "Device:C_Polarized_Small_US") (at 61.595 145.415 0) (unit 1)
     (in_bom yes) (on_board yes)
-    (property "Reference" "C11" (id 0) (at 64.77 143.7131 0)
+    (property "Reference" "C12" (id 0) (at 64.77 143.7131 0)
       (effects (font (size 1.27 1.27)) (justify left))
     )
@@
   (symbol (lib_id "power:+5V") (at 33.02 63.5 0) (unit 1)
     (in_bom yes) (on_board yes) (fields_autoplaced)
-    (property "Reference" "#PWR021" (id 0) (at 33.02 67.31 0)
+    (property "Reference" "#PWR022" (id 0) (at 33.02 67.31 0)
       (effects (font (size 1.27 1.27)) hide)
     )
@@
   (symbol (lib_id "Device:C") (at 182.88 93.98 0) (unit 1)
     (in_bom yes) (on_board yes) (fields_autoplaced)
-    (property "Reference" "C17" (id 0) (at 186.69 92.7099 0)
+    (property "Reference" "C18" (id 0) (at 186.69 92.7099 0)
       (effects (font (size 1.27 1.27)) (justify left))
     )
@@
   (symbol (lib_id "power:+5V") (at 52.705 137.795 0) (unit 1)
     (in_bom yes) (on_board yes) (fields_autoplaced)
-    (property "Reference" "#PWR023" (id 0) (at 52.705 141.605 0)
-      (effects (font (size 1.27 1.27)) hide)
-    )
+    (property "Reference" "#PWR024" (id 0) (at 52.705 141.605 0)
+      (effects (font (size 1.27 1.27)) hide)
+    )
