File: Embebidos/USB_UART.kicad_sch (KiCad schematic)
At the start: 9 parts, among them Q1 BC847, Q2 BC847

Commit message: huellass
Parts:
- removed J1: ~, symbol Connector:USB_B_Micro
- added J1: USB_A, Connector_USB:USB_A_CNCTech_1001-011-01101_Horizontal, symbol Connector:USB_A
- C5, C6, C7: footprint (none) -> Capacitor_SMD:C_0805_2012Metric_Pad1.18x1.45mm_HandSolder
- Q1, Q2: footprint Package_TO_SOT_SMD:SOT-23 -> BC847:SOT23
- R13, R14: footprint (none) -> Resistor_SMD:R_0805_2012Metric_Pad1.20x1.40mm_HandSolder
- U1: footprint (none) -> CP2104:QFN50P400X400X80-25N
Connections:
- net D+: now also J1.3 (D+)
- net D-: now also J1.2 (D-)
- net GND: now also J1.4 (GND), J1.5 (Shield)
- net VBUS: now also J1.1 (VBUS)
Changed lines of the file:
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@@
   (junction (at 91.44 116.84) (diameter 0) (color 0 0 0 0)
   )
-  (no_connect (at 90.17 96.52))
+  (no_connect (at 86.36 96.52))
   (no_connect (at 143.51 106.68))
   (no_connect (at 143.51 109.22))
@@
     (pin "1")
   )
-  (symbol (lib_id "Connector:USB_B_Micro") (at 82.55 91.44 0) (unit 1)
+  (symbol (lib_id "Connector:USB_A") (at 82.55 91.44 0) (unit 1)
     (in_bom yes) (on_board yes) (fields_autoplaced)
     (property "Reference" "J1" (id 0) (at 82.55 78.74 0))
-    (property "Value" "~" (id 1) (at 82.55 81.28 0))
-    (property "Footprint" "" (id 2) (at 86.36 92.71 0)
-      (effects (font (size 1.27 1.27)) hide)
-    )
-    (property "Datasheet" "~" (id 3) (at 86.36 92.71 0)
+    (property "Value" "USB_A" (id 1) (at 82.55 81.28 0))
+    (property "Footprint" "Connector_USB:USB_A_CNCTech_1001-011-01101_Horizontal" (id 2) (at 86.36 92.71 0)
+      (effects (font (size 1.27 1.27)) hide)
+    )
+    (property "Datasheet" " ~" (id 3) (at 86.36 92.71 0)
       (effects (font (size 1.27 1.27)) hide)
     )
@@
     (pin "4")
     (pin "5")
-    (pin "6")
   )
   (symbol (lib_id "power:+3.3V") (at 91.44 116.84 0) (unit 1)
@@
       (effects (font (size 1.27 1.27)) (justify left))
     )
-    (property "Footprint" "Package_TO_SOT_SMD:SOT-23" (id 2) (at 201.93 92.075 0)
+    (property "Footprint" "BC847:SOT23" (id 2) (at 201.93 92.075 0)
       (effects (font (size 1.27 1.27) italic) (justify left) hide)
     )
@@
     (property "Reference" "R13" (id 0) (at 184.15 83.82 90))
     (property "Value" "10k" (id 1) (at 184.15 86.36 90))
-    (property "Footprint" "" (id 2) (at 184.15 91.948 90)
+    (property "Footprint" "Resistor_SMD:R_0805_2012Metric_Pad1.20x1.40mm_HandSolder" (id 2) (at 184.15 91.948 90)
       (effects (font (size 1.27 1.27)) hide)
     )
@@
       (effects (font (size 1.27 1.27)) (justify left))
     )
-    (property "Footprint" "" (id 2) (at 98.7552 127 0)
+    (property "Footprint" "Capacitor_SMD:C_0805_2012Metric_Pad1.18x1.45mm_HandSolder" (id 2) (at 98.7552 127 0)
       (effects (font (size 1.27 1.27)) hide)
     )
@@
       (effects (font (size 1.27 1.27)) (justify left))
     )
-    (property "Footprint" "" (id 2) (at 160.02 148.59 0)
+    (property "Footprint" "CP2104:QFN50P400X400X80-25N" (id 2) (at 160.02 148.59 0)
       (effects (font (size 1.27 1.27)) (justify left) hide)
     )
@@
       (effects (font (size 1.27 1.27)) (justify left))
     )
-    (property "Footprint" "Package_TO_SOT_SMD:SOT-23" (id 2) (at 201.93 116.205 0)
+    (property "Footprint" "BC847:SOT23" (id 2) (at 201.93 116.205 0)
       (effects (font (size 1.27 1.27) italic) (justify left) hide)
     )
@@
       (effects (font (size 1.27 1.27)) (justify left))
     )
-    (property "Footprint" "" (id 2) (at 87.3252 127 0)
+    (property "Footprint" "Capacitor_SMD:C_0805_2012Metric_Pad1.18x1.45mm_HandSolder" (id 2) (at 87.3252 127 0)
       (effects (font (size 1.27 1.27)) hide)
     )
@@
     (property "Reference" "R14" (id 0) (at 184.15 107.95 90))
     (property "Value" "10k" (id 1) (at 184.15 110.49 90))
-    (property "Footprint" "" (id 2) (at 184.15 116.078 90)
+    (property "Footprint" "Resistor_SMD:R_0805_2012Metric_Pad1.20x1.40mm_HandSolder" (id 2) (at 184.15 116.078 90)
       (effects (font (size 1.27 1.27)) hide)
     )
@@
       (effects (font (size 1.27 1.27)) (justify left))
     )
-    (property "Footprint" "" (id 2) (at 112.7252 128.27 0)
-      (effects (font (size 1.27 1.27)) hide)
-    )
+    (property "Footprint" "Capacitor_SMD:C_0805_2012Metric_Pad1.18x1.45mm_HandSolder" (id 2) (at 112.7252 128.27 0)
+      (effects (font (size 1.27 1.27)) hide)
+    )

Commit message: .
Connections:
- no-connect marks 12 -> 11
Changed lines of the file:
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@@
   (junction (at 91.44 116.84) (diameter 0) (color 0 0 0 0)
   )
-  (no_connect (at 86.36 96.52))
   (no_connect (at 143.51 106.68))
   (no_connect (at 143.51 109.22))
