File: Embebidos/conn_sensores.kicad_sch (KiCad schematic)
At the start: 2 parts, among them J10 Conn_01x08, J9 Conn_01x05

Commit message: huellass
Parts:
- removed J9: Conn_01x05, symbol Connector_Generic:Conn_01x05
- added J9: Conn_02x06_Counter_Clockwise, HUELLA SIM800L:sim800l, symbol Connector_Generic:Conn_02x06_Counter_Clockwise
- J10: footprint (none) -> Connector_PinHeader_2.54mm:PinHeader_1x08_P2.54mm_Vertical
Connections:
- net 4.1V: now also J9.2 (Pin_2)
- net GND: now also J9.6 (Pin_6)
- net RXSIM: now also J9.5 (Pin_5)
- net TXSIM: now also J9.4 (Pin_4)
- no-connect marks 3 -> 10
Changed lines of the file:
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@@
   (paper "A4")
   (no_connect (at 97.79 64.77))
+  (no_connect (at 86.36 26.67))
+  (no_connect (at 86.36 31.75))
+  (no_connect (at 99.06 29.21))
+  (no_connect (at 99.06 34.29))
+  (no_connect (at 99.06 36.83))
+  (no_connect (at 99.06 31.75))
+  (no_connect (at 99.06 39.37))
+  (no_connect (at 99.06 26.67))
   (no_connect (at 97.79 69.85))
-  (no_connect (at 97.79 30.48))
-  (global_label "4.1V" (shape output) (at 97.79 27.94 0) (fields_autoplaced)
-    (effects (font (size 1.27 1.27)) (justify left))
-    (property "Intersheet References" "${INTERSHEET_REFS}" (id 0) (at 104.3155 27.8606 0)
-      (effects (font (size 1.27 1.27)) (justify left) hide)
+  (wire (pts (xy 86.36 39.37) (xy 83.82 39.37))
+    (stroke (width 0) (type default) (color 0 0 0 0))
+  )
+  (wire (pts (xy 86.36 36.83) (xy 83.82 36.83))
+    (stroke (width 0) (type default) (color 0 0 0 0))
+  )
+  (wire (pts (xy 86.36 29.21) (xy 83.82 29.21))
+    (stroke (width 0) (type default) (color 0 0 0 0))
+  )
+  (wire (pts (xy 86.36 34.29) (xy 83.82 34.29))
+    (stroke (width 0) (type default) (color 0 0 0 0))
+  )
+  (global_label "4.1V" (shape output) (at 83.82 29.21 180) (fields_autoplaced)
+    (effects (font (size 1.27 1.27)) (justify right))
+    (property "Intersheet References" "${INTERSHEET_REFS}" (id 0) (at 77.2945 29.1306 0)
+      (effects (font (size 1.27 1.27)) (justify right) hide)
     )
   )
@@
     (effects (font (size 1.27 1.27)) (justify left))
   )
-  (hierarchical_label "TXSIM" (shape bidirectional) (at 97.79 33.02 0)
+  (hierarchical_label "MISO_RFID" (shape input) (at 97.79 62.23 0)
     (effects (font (size 1.27 1.27)) (justify left))
   )
-  (hierarchical_label "RXSIM" (shape bidirectional) (at 97.79 35.56 0)
-    (effects (font (size 1.27 1.27)) (justify left))
+  (hierarchical_label "TXSIM" (shape bidirectional) (at 83.82 34.29 180)
+    (effects (font (size 1.27 1.27)) (justify right))
   )
-  (hierarchical_label "MISO_RFID" (shape input) (at 97.79 62.23 0)
-    (effects (font (size 1.27 1.27)) (justify left))
+  (hierarchical_label "RXSIM" (shape bidirectional) (at 83.82 36.83 180)
+    (effects (font (size 1.27 1.27)) (justify right))
   )
   (hierarchical_label "SCK_RFID" (shape input) (at 97.79 57.15 0)
@@
   (hierarchical_label "MOSI_RFID" (shape input) (at 97.79 59.69 0)
     (effects (font (size 1.27 1.27)) (justify left))
+  )
+  (symbol (lib_id "power:GND") (at 83.82 39.37 270) (unit 1)
+    (in_bom yes) (on_board yes)
+    (property "Reference" "#PWR044" (id 0) (at 77.47 39.37 0)
+      (effects (font (size 1.27 1.27)) hide)
+    )
+    (property "Value" "GND" (id 1) (at 76.2 39.37 90)
+      (effects (font (size 1.27 1.27)) (justify left))
+    )
+    (property "Footprint" "" (id 2) (at 83.82 39.37 0)
+      (effects (font (size 1.27 1.27)) hide)
+    )
+    (property "Datasheet" "" (id 3) (at 83.82 39.37 0)
+      (effects (font (size 1.27 1.27)) hide)
+    )
+    (pin "1")
+  )
+  (symbol (lib_id "Connector_Generic:Conn_02x06_Counter_Clockwise") (at 91.44 31.75 0) (unit 1)
+    (in_bom yes) (on_board yes) (fields_autoplaced)
+    (property "Reference" "J9" (id 0) (at 92.71 20.32 0))
+    (property "Value" "Conn_02x06_Counter_Clockwise" (id 1) (at 92.71 22.86 0))
+    (property "Footprint" "HUELLA SIM800L:sim800l" (id 2) (at 91.44 31.75 0)
+      (effects (font (size 1.27 1.27)) hide)
+    )
+    (property "Datasheet" "~" (id 3) (at 91.44 31.75 0)
+      (effects (font (size 1.27 1.27)) hide)
+    )
+    (pin "1")
+    (pin "10")
+    (pin "11")
+    (pin "12")
+    (pin "2")
+    (pin "3")
+    (pin "4")
+    (pin "5")
+    (pin "6")
+    (pin "7")
+    (pin "8")
+    (pin "9")
   )
   (symbol (lib_id "power:+3.3V") (at 97.79 72.39 270) (mirror x) (unit 1)
@@
     (pin "1")
   )
-  (symbol (lib_id "Connector_Generic:Conn_01x05") (at 92.71 33.02 0) (mirror y) (unit 1)
-    (in_bom yes) (on_board yes) (fields_autoplaced)
-    (property "Reference" "J9" (id 0) (at 90.17 31.7499 0)
-      (effects (font (size 1.27 1.27)) (justify left))
-    )
-    (property "Value" "Conn_01x05" (id 1) (at 90.17 34.2899 0)
-      (effects (font (size 1.27 1.27)) (justify left))
-    )
-    (property "Footprint" "" (id 2) (at 92.71 33.02 0)
-      (effects (font (size 1.27 1.27)) hide)
-    )
-    (property "Datasheet" "~" (id 3) (at 92.71 33.02 0)
-      (effects (font (size 1.27 1.27)) hide)
-    )
-    (pin "1")
-    (pin "2")
-    (pin "3")
-    (pin "4")
-    (pin "5")
-  )
   (symbol (lib_id "Connector_Generic:Conn_01x08") (at 92.71 62.23 0) (mirror y) (unit 1)
     (in_bom yes) (on_board yes) (fields_autoplaced)
-    (property "Reference" "J10" (id 0) (at 90.17 62.2299 0)
-      (effects (font (size 1.27 1.27)) (justify left))
-    )
-    (property "Value" "Conn_01x08" (id 1) (at 90.17 64.7699 0)
-      (effects (font (size 1.27 1.27)) (justify left))
-    )
-    (property "Footprint" "" (id 2) (at 92.71 62.23 0)
+    (property "Reference" "J10" (id 0) (at 92.71 48.26 0))
+    (property "Value" "Conn_01x08" (id 1) (at 92.71 50.8 0))
+    (property "Footprint" "Connector_PinHeader_2.54mm:PinHeader_1x08_P2.54mm_Vertical" (id 2) (at 92.71 62.23 0)
       (effects (font (size 1.27 1.27)) hide)
     )
@@
     (pin "8")
   )
-  (symbol (lib_id "power:GND") (at 97.79 38.1 90) (mirror x) (unit 1)
-    (in_bom yes) (on_board yes) (fields_autoplaced)
-    (property "Reference" "#PWR044" (id 0) (at 104.14 38.1 0)
-      (effects (font (size 1.27 1.27)) hide)
-    )
-    (property "Value" "GND" (id 1) (at 101.6 38.0999 90)
-      (effects (font (size 1.27 1.27)) (justify right))
-    )
-    (property "Footprint" "" (id 2) (at 97.79 38.1 0)
-      (effects (font (size 1.27 1.27)) hide)
-    )
-    (property "Datasheet" "" (id 3) (at 97.79 38.1 0)
-      (effects (font (size 1.27 1.27)) hide)
-    )
-    (pin "1")
-  )
 )

Commit message: Anotaciones
Parts:
- renumbered J9 to J5, J10 to J6
Changed lines of the file:
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@@
   (symbol (lib_id "Connector_Generic:Conn_02x06_Counter_Clockwise") (at 91.44 31.75 0) (unit 1)
     (in_bom yes) (on_board yes) (fields_autoplaced)
-    (property "Reference" "J9" (id 0) (at 92.71 20.32 0))
+    (property "Reference" "J5" (id 0) (at 92.71 20.32 0))
     (property "Value" "Conn_02x06_Counter_Clockwise" (id 1) (at 92.71 22.86 0))
     (property "Footprint" "HUELLA SIM800L:sim800l" (id 2) (at 91.44 31.75 0)
@@
   (symbol (lib_id "Connector_Generic:Conn_01x08") (at 92.71 62.23 0) (mirror y) (unit 1)
     (in_bom yes) (on_board yes) (fields_autoplaced)
-    (property "Reference" "J10" (id 0) (at 92.71 48.26 0))
+    (property "Reference" "J6" (id 0) (at 92.71 48.26 0))
     (property "Value" "Conn_01x08" (id 1) (at 92.71 50.8 0))
     (property "Footprint" "Connector_PinHeader_2.54mm:PinHeader_1x08_P2.54mm_Vertical" (id 2) (at 92.71 62.23 0)

Commit message: .
Parts:
- added J5: Conn_01x04, symbol Connector_Generic:Conn_01x04
- renumbered J5 to J6, J6 to J7
Connections:
- net +3.3V: now also J5.1 (Pin_1)
- net GND: now also J5.4 (Pin_4)
- new net RXGPS: J5.2 (Pin_2)
- new net TXGPS: J5.3 (Pin_3)
Changed lines of the file:
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@@
+    (stroke (width 0) (type default) (color 0 0 0 0))
+  )
+  (wire (pts (xy 85.09 87.63) (xy 81.28 87.63))
     (stroke (width 0) (type default) (color 0 0 0 0))
   )
@@
   )
   (wire (pts (xy 86.36 29.21) (xy 83.82 29.21))
+    (stroke (width 0) (type default) (color 0 0 0 0))
+  )
+  (wire (pts (xy 78.74 92.71) (xy 85.09 92.71))
+    (stroke (width 0) (type default) (color 0 0 0 0))
+  )
+  (wire (pts (xy 81.28 87.63) (xy 81.28 86.36))
+    (stroke (width 0) (type default) (color 0 0 0 0))
+  )
+  (wire (pts (xy 85.09 95.25) (xy 81.28 95.25))
+    (stroke (width 0) (type default) (color 0 0 0 0))
+  )
+  (wire (pts (xy 78.74 90.17) (xy 85.09 90.17))
+    (stroke (width 0) (type default) (color 0 0 0 0))
+  )
+  (wire (pts (xy 81.28 95.25) (xy 81.28 96.52))
     (stroke (width 0) (type default) (color 0 0 0 0))
   )
@@
     (effects (font (size 1.27 1.27)) (justify left))
   )
+  (hierarchical_label "TXGPS" (shape bidirectional) (at 78.74 92.71 180)
+    (effects (font (size 1.27 1.27)) (justify right))
+  )
   (hierarchical_label "TXSIM" (shape bidirectional) (at 83.82 34.29 180)
     (effects (font (size 1.27 1.27)) (justify right))
@@
     (effects (font (size 1.27 1.27)) (justify left))
   )
+  (hierarchical_label "RXGPS" (shape bidirectional) (at 78.74 90.17 180)
+    (effects (font (size 1.27 1.27)) (justify right))
+  )
   (hierarchical_label "MOSI_RFID" (shape input) (at 97.79 59.69 0)
     (effects (font (size 1.27 1.27)) (justify left))
@@
   (symbol (lib_id "power:GND") (at 83.82 39.37 270) (unit 1)
     (in_bom yes) (on_board yes)
-    (property "Reference" "#PWR044" (id 0) (at 77.47 39.37 0)
+    (property "Reference" "#PWR046" (id 0) (at 77.47 39.37 0)
       (effects (font (size 1.27 1.27)) hide)
     )
@@
   (symbol (lib_id "Connector_Generic:Conn_02x06_Counter_Clockwise") (at 91.44 31.75 0) (unit 1)
     (in_bom yes) (on_board yes) (fields_autoplaced)
-    (property "Reference" "J5" (id 0) (at 92.71 20.32 0))
+    (property "Reference" "J6" (id 0) (at 92.71 20.32 0))
     (property "Value" "Conn_02x06_Counter_Clockwise" (id 1) (at 92.71 22.86 0))
     (property "Footprint" "HUELLA SIM800L:sim800l" (id 2) (at 91.44 31.75 0)
@@
     (pin "9")
   )
+  (symbol (lib_id "Connector_Generic:Conn_01x04") (at 90.17 90.17 0) (unit 1)
+    (in_bom yes) (on_board yes) (fields_autoplaced)
+    (property "Reference" "J5" (id 0) (at 92.71 90.1699 0)
+      (effects (font (size 1.27 1.27)) (justify left))
+    )
+    (property "Value" "Conn_01x04" (id 1) (at 92.71 92.7099 0)
+      (effects (font (size 1.27 1.27)) (justify left))
+    )
+    (property "Footprint" "" (id 2) (at 90.17 90.17 0)
+      (effects (font (size 1.27 1.27)) hide)
+    )
+    (property "Datasheet" "~" (id 3) (at 90.17 90.17 0)
+      (effects (font (size 1.27 1.27)) hide)
+    )
+    (pin "1")
+    (pin "2")
+    (pin "3")
+    (pin "4")
+  )
   (symbol (lib_id "power:+3.3V") (at 97.79 72.39 270) (mirror x) (unit 1)
     (in_bom yes) (on_board yes) (fields_autoplaced)
-    (property "Reference" "#PWR046" (id 0) (at 93.98 72.39 0)
+    (property "Reference" "#PWR048" (id 0) (at 93.98 72.39 0)
       (effects (font (size 1.27 1.27)) hide)
     )
@@
     (pin "1")
   )
+  (symbol (lib_id "power:GND") (at 81.28 96.52 0) (unit 1)
+    (in_bom yes) (on_board yes) (fields_autoplaced)
+    (property "Reference" "#PWR045" (id 0) (at 81.28 102.87 0)
+      (effects (font (size 1.27 1.27)) hide)
+    )
+    (property "Value" "GND" (id 1) (at 81.28 101.6 0))
+    (property "Footprint" "" (id 2) (at 81.28 96.52 0)
+      (effects (font (size 1.27 1.27)) hide)
+    )
+    (property "Datasheet" "" (id 3) (at 81.28 96.52 0)
+      (effects (font (size 1.27 1.27)) hide)
+    )
+    (pin "1")
+  )
+  (symbol (lib_id "power:+3.3V") (at 81.28 86.36 0) (unit 1)
+    (in_bom yes) (on_board yes)
+    (property "Reference" "#PWR044" (id 0) (at 81.28 90.17 0)
+      (effects (font (size 1.27 1.27)) hide)
+    )
+    (property "Value" "+3.3V" (id 1) (at 81.661 81.9658 0))
+    (property "Footprint" "" (id 2) (at 81.28 86.36 0)
+      (effects (font (size 1.27 1.27)) hide)
+    )
+    (property "Datasheet" "" (id 3) (at 81.28 86.36 0)
+      (effects (font (size 1.27 1.27)) hide)
+    )
+    (pin "1")
+  )
   (symbol (lib_id "power:GND") (at 97.79 67.31 90) (mirror x) (unit 1)
     (in_bom yes) (on_board yes) (fields_autoplaced)
-    (property "Reference" "#PWR045" (id 0) (at 104.14 67.31 0)
+    (property "Reference" "#PWR047" (id 0) (at 104.14 67.31 0)
       (effects (font (size 1.27 1.27)) hide)
     )
@@
   (symbol (lib_id "Connector_Generic:Conn_01x08") (at 92.71 62.23 0) (mirror y) (unit 1)
     (in_bom yes) (on_board yes) (fields_autoplaced)
-    (property "Reference" "J6" (id 0) (at 92.71 48.26 0))
+    (property "Reference" "J7" (id 0) (at 92.71 48.26 0))
     (property "Value" "Conn_01x08" (id 1) (at 92.71 50.8 0))
     (property "Footprint" "Connector_PinHeader_2.54mm:PinHeader_1x08_P2.54mm_Vertical" (id 2) (at 92.71 62.23 0)

Commit message: .
Parts:
- J5: footprint (none) -> Connector_PinHeader_2.54mm:PinHeader_1x04_P2.54mm_Vertical
Connections:
- net +3.3V: no longer J7.8 (Pin_8)
- new net 3.3Vop2: J7.8 (Pin_8)
Changed lines of the file:
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@@
+    (stroke (width 0) (type default) (color 0 0 0 0))
+  )
+  (wire (pts (xy 97.79 72.39) (xy 99.06 72.39))
     (stroke (width 0) (type default) (color 0 0 0 0))
   )
@@
   (wire (pts (xy 86.36 34.29) (xy 83.82 34.29))
     (stroke (width 0) (type default) (color 0 0 0 0))
+  )
+  (global_label "3.3Vop2" (shape input) (at 99.06 72.39 0) (fields_autoplaced)
+    (effects (font (size 1.27 1.27)) (justify left))
+    (property "Intersheet References" "${INTERSHEET_REFS}" (id 0) (at 109.0931 72.3106 0)
+      (effects (font (size 1.27 1.27)) (justify left) hide)
+    )
   )
   (global_label "4.1V" (shape output) (at 83.82 29.21 180) (fields_autoplaced)
@@
       (effects (font (size 1.27 1.27)) (justify left))
     )
-    (property "Footprint" "" (id 2) (at 90.17 90.17 0)
+    (property "Footprint" "Connector_PinHeader_2.54mm:PinHeader_1x04_P2.54mm_Vertical" (id 2) (at 90.17 90.17 0)
       (effects (font (size 1.27 1.27)) hide)
     )
@@
     (pin "4")
   )
-  (symbol (lib_id "power:+3.3V") (at 97.79 72.39 270) (mirror x) (unit 1)
-    (in_bom yes) (on_board yes) (fields_autoplaced)
-    (property "Reference" "#PWR048" (id 0) (at 93.98 72.39 0)
-      (effects (font (size 1.27 1.27)) hide)
-    )
-    (property "Value" "+3.3V" (id 1) (at 101.6 72.3899 90)
-      (effects (font (size 1.27 1.27)) (justify left))
-    )
-    (property "Footprint" "" (id 2) (at 97.79 72.39 0)
-      (effects (font (size 1.27 1.27)) hide)
-    )
-    (property "Datasheet" "" (id 3) (at 97.79 72.39 0)
-      (effects (font (size 1.27 1.27)) hide)
-    )
-    (pin "1")
-  )
   (symbol (lib_id "power:GND") (at 81.28 96.52 0) (unit 1)
