File: Embebidos/_autosave-EsquemaGeneral.kicad_pcb (KiCad board)
At the start: 2 copper layers, 100 x 99.9 mm, 79 parts, among them IC1 ESP32-WROVER-B__8MB_, J1 USB_A, J2 Conn_01x02, J3 RJ45, J4 RJ45, J5 Conn_02x06_Counter_Clockwise, J6 Conn_01x08, J7 Conn_01x04, Q1 BC847, Q2 BC847, Q3 BSS138, Q4 DMP3056LSDQ-13, Q5 BSS138, Q6 DMP3056LSDQ-13, SW1 SW_Reset, SW2 SW_Boot, U2 LM358, U3 SPX3819M5-L-3-3, U4 MIC29302WU, U5 MIC5219-3.3YM5

Commit message: aa
Changed lines of the file:
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@@
     (property "Sheetfile" "USB_UART.kicad_sch")
     (property "Sheetname" "USB_UART")
-    (clearance 0.1)
+    (clearance 0.15)
     (attr smd)
     (fp_text reference "U1" (at -0.25427 -3.43257 90) (layer "F.SilkS")
@@
   (segment (start 176.8754 125.4346) (end 176.8754 58.2328) (width 0.6) (layer "B.Cu") (net 47))
   (segment (start 167.94 134.37) (end 176.8754 125.4346) (width 0.6) (layer "B.Cu") (net 47))
-  (segment (start 121.81 58.1202) (end 121.81 53.14) (width 0.25) (layer "F.Cu") (net 60))
-  (segment (start 121.07 58.8602) (end 121.81 58.1202) (width 0.25) (layer "F.Cu") (net 60))
-  (segment (start 121.07 59.44) (end 121.07 58.8602) (width 0.25) (layer "F.Cu") (net 60))
+  (segment (start 121.07 59.44) (end 121.07 53.88) (width 0.25) (layer "F.Cu") (net 60))
+  (segment (start 121.07 53.88) (end 121.81 53.14) (width 0.25) (layer "F.Cu") (net 60))
   (segment (start 98.38 55.38) (end 104.36 55.38) (width 0.6) (layer "F.Cu") (net 61))
   (segment (start 104.36 55.38) (end 107.36 52.38) (width 0.6) (layer "F.Cu") (net 61))
